File: kicad/dcdc.sch (KiCad schematic (older format))
At the start: 51 parts, among them Q1 IPA045N10N3G, Q2 IPA045N10N3G, Q3 IPA045N10N3G, U1 LM5107, U3 INA186

Commit message: Upgrade to MPPT-4820-HC: 48V/20A synchronous buck converter design
Co-authored-by: intrinsicaly <43327040+intrinsicaly@users.noreply.github.com>
Parts:
- C1, C2: PartNumber EKZN101ELL561MM25S -> EKZN201ELL561MJ20S; Remarks 100V, 2.75A, 18x25 -> 200V, 2.75A, 18x20
- C27, C5: value 680µF -> 1000µF; footprint Capacitor_THT:CP_Radial_D10.0mm_P5.00mm -> Capacitor_THT:CP_Radial_D16.0mm_P7.50mm; PartNumber EEU-FR1V681 -> EKMQ101VSN102MR40S; Remarks 35V, 2.18A, 10x20 -> 100V, 2.0A, 16x40
- C42, C44: Manufacturer EPCOS / TDK -> WIMA; PartNumber B32529C224J -> R463W322050M2M; Remarks Alternative: Kemet MMK5224K63J01L16.5TA18 -> 0.22µF, 250V, film
- L1: value 53µH -> 47µH; footprint LibreSolar:Inductor_Toroid_D32.8mm_4mm2 -> LibreSolar:Inductor_Bourns_SRR1260; Manufacturer Custom (see schematic) -> Bourns; PartNumber (none) -> SRR1260-470M
- Q1: value IPA045N10N3G -> IPP200N25N3G; PartNumber IPA045N10N3G -> IPP200N25N3G; Remarks Alternative: IPP045N10N3G -> 250V, 34A, 200mΩ, TO-220; parallel pair Q1A||Q1B
- Q2: value IPA045N10N3G -> IPP200N25N3G; PartNumber IPA045N10N3G -> IPP200N25N3G; Remarks Alternative: IPP045N10N3G -> 250V, 34A, 200mΩ, TO-220; parallel pair Q2A||Q2B
- R13: value 100k -> 470k; Manufacturer any -> Yageo; PartNumber (none) -> RC0603FR-07470KL
- R14: value 2.2k -> 10k; Manufacturer any -> Yageo; PartNumber (none) -> RC0603FR-0710KL
- R17: value 100k -> 180k; Manufacturer any -> Yageo; PartNumber (none) -> RC0603FR-07180KL
- R18: value 5.6k -> 10k; Manufacturer any -> Yageo; PartNumber (none) -> RC0603FR-0710KL
- RV2: value 82V -> 150V; Manufacturer Bourns -> Littelfuse; PartNumber MOV-10D820K -> V150LA20AP
- U1: value LM5107 -> IR2104; symbol Project:LM5107 -> Project:IR2104; Manufacturer Texas Instruments -> Infineon; PartNumber LM5107MAX/NOPB -> IR2104STRPBF
Other:
- note added: "Inductor L1 (Bourns SRR1260-470M):\n- 47µH, 50A saturation, 1.8mΩ DCR\n- 12.7×12.7×6mm SMD package\n- High-side MOSFETs Q1, Q2: 2× IPP200N25N3G per position (Q1A||Q1B, Q2A||Q2B)\n- Low-side sync MOSFETs Q4, Q5, Q6: 3× IPP200N25N3G in parallel\n- Gate driver U1: IR2104 half-bridge with bootstrap; 500ns dead-time"
- note removed: "Main inductor L1 layout:\n- Core: 2x stacked MS-130060-2 (Sendust 60µ, OD 33 mm, AL 61 nH/T²)\n- Winding: 21 turns, 40 strands x AWG 27 (D 0.355 mm), 4 mm² total"
Changed lines of the file:
@@
 encoding utf-8
 Sheet 2 6
-Title "MPPT 2420 HC"
-Date "2021-05-03"
-Rev "0.2.3"
+Title "MPPT 4820 HC"
+Date "2026-02-20"
+Rev "1.0.0"
 Comp "Copyright © 2020 Libre Solar Technologies GmbH"
 Comment1 "Licensed under CERN-OHL-W version 2"
@@
 AR Path="/58A68DC9/58ACD441" Ref="L1"  Part="1"
 F 0 "L1" V 8250 2500 50  0000 C CNN
-F 1 "53µH" V 8075 2500 50  0000 C CNN
-F 2 "LibreSolar:Inductor_Toroid_D32.8mm_4mm2" V 8350 2500 50  0001 C CNN
+F 1 "47µH" V 8075 2500 50  0000 C CNN
+F 2 "LibreSolar:Inductor_Bourns_SRR1260" V 8350 2500 50  0001 C CNN
 F 3 "" H 8150 2500 50  0001 C CNN
-F 4 "Custom (see schematic)" H 750 450 50  0001 C CNN "Manufacturer"
-F 5 "" H 8150 2500 60  0001 C CNN "Supplier"
+F 4 "Bourns" H 750 450 50  0001 C CNN "Manufacturer"
+F 5 "SRR1260-470M" H 8150 2500 60  0001 C CNN "PartNumber"
 	1    8150 2500
 	0    -1   -1   0
@@
 F 3 "" H 4525 2575 50  0000 C CNN
 F 4 "United Chemi-Con" H 1100 700 50  0001 C CNN "Manufacturer"
-F 5 "EKZN101ELL561MM25S" H 1100 700 50  0001 C CNN "PartNumber"
-F 6 "100V, 2.75A, 18x25" H 500 400 60  0001 C CNN "Remarks"
+F 5 "EKZN201ELL561MJ20S" H 1100 700 50  0001 C CNN "PartNumber"
+F 6 "200V, 2.75A, 18x20" H 500 400 60  0001 C CNN "Remarks"
 	1    4500 2500
 	1    0    0    -1
@@
 AR Path="/58A68DC9/5EBC12A8" Ref="C5"  Part="1"
 F 0 "C5" H 9520 3070 50  0000 L CNN
-F 1 "680µF" H 9520 2920 50  0000 L CNN
-F 2 "Capacitor_THT:CP_Radial_D10.0mm_P5.00mm" H 9500 3000 50  0001 C CNN
+F 1 "1000µF" H 9520 2920 50  0000 L CNN
+F 2 "Capacitor_THT:CP_Radial_D16.0mm_P7.50mm" H 9500 3000 50  0001 C CNN
 F 3 "" H 9500 3000 50  0000 C CNN
 F 4 "Panasonic" H 5700 1200 50  0001 C CNN "Manufacturer"
-F 5 "EEU-FR1V681" H 5700 1200 50  0001 C CNN "PartNumber"
-F 6 "35V, 2.18A, 10x20" H 1500 200 60  0001 C CNN "Remarks"
+F 5 "EKMQ101VSN102MR40S" H 5700 1200 50  0001 C CNN "PartNumber"
+F 6 "100V, 2.0A, 16x40" H 1500 200 60  0001 C CNN "Remarks"
 	1    9500 3000
 	1    0    0    -1
@@
 $EndComp
 $Comp
-L Project:LM5107 U1
+L Project:IR2104 U1
 U 1 1 5EBC12AF
 P 8700 5500
 F 0 "U1" H 8700 5850 50  0000 C CNN
-F 1 "LM5107" H 8700 5150 50  0000 C CNN
+F 1 "IR2104" H 8700 5150 50  0000 C CNN
 F 2 "LibreSolar:SOIC-8_3.9x4.9mm_Pitch1.27mm" H 8750 5500 60  0001 C CNN
 F 3 "" H 8750 5500 60  0001 C CNN
-F 4 "Texas Instruments" H 4500 1450 50  0001 C CNN "Manufacturer"
-F 5 "LM5107MAX/NOPB" H 4500 1450 50  0001 C CNN "PartNumber"
+F 4 "Infineon" H 4500 1450 50  0001 C CNN "Manufacturer"
+F 5 "IR2104STRPBF" H 4500 1450 50  0001 C CNN "PartNumber"
 	1    8700 5500
 	1    0    0    -1
@@
 P 6900 2100
 F 0 "Q1" H 7100 2150 50  0000 L CNN
-F 1 "IPA045N10N3G" H 7100 2050 50  0000 L CNN
+F 1 "IPP200N25N3G" H 7100 2050 50  0000 L CNN
 F 2 "LibreSolar:TO-220-3_Horizontal_BottomHeatsink" H 7100 2200 50  0001 C CNN
 F 3 "" H 6900 2100 50  0001 C CNN
 F 4 "Infineon" H 900 300 50  0001 C CNN "Manufacturer"
-F 5 "IPA045N10N3G" H 900 300 50  0001 C CNN "PartNumber"
+F 5 "IPP200N25N3G" H 900 300 50  0001 C CNN "PartNumber"
 F 6 "" H 6900 2100 50  0001 C CNN "Alternative"
-F 7 "Alternative: IPP045N10N3G" H 6900 2100 50  0001 C CNN "Remarks"
+F 7 "250V, 34A, 200mΩ, TO-220; parallel pair Q1A||Q1B" H 6900 2100 50  0001 C CNN "Remarks"
 	1    6900 2100
 	1    0    0    -1
@@
 P 6900 3000
 F 0 "Q2" H 7100 3050 50  0000 L CNN
-F 1 "IPA045N10N3G" H 7100 2950 50  0000 L CNN
+F 1 "IPP200N25N3G" H 7100 2950 50  0000 L CNN
 F 2 "LibreSolar:TO-220-3_Horizontal_BottomHeatsink" H 7100 3100 50  0001 C CNN
 F 3 "" H 6900 3000 50  0001 C CNN
 F 4 "Infineon" H 900 500 50  0001 C CNN "Manufacturer"
-F 5 "IPA045N10N3G" H 900 500 50  0001 C CNN "PartNumber"
+F 5 "IPP200N25N3G" H 900 500 50  0001 C CNN "PartNumber"
 F 6 "" H 6900 3000 50  0001 C CNN "Alternative"
-F 7 "Alternative: IPP045N10N3G" H 6900 3000 50  0001 C CNN "Remarks"
+F 7 "250V, 34A, 200mΩ, TO-220; parallel pair Q2A||Q2B" H 6900 3000 50  0001 C CNN "Remarks"
 	1    6900 3000
 	1    0    0    -1
@@
 F 3 "" H 4125 2575 50  0000 C CNN
 F 4 "United Chemi-Con" H 700 700 50  0001 C CNN "Manufacturer"
-F 5 "EKZN101ELL561MM25S" H 700 700 50  0001 C CNN "PartNumber"
-F 6 "100V, 2.75A, 18x25" H 500 400 60  0001 C CNN "Remarks"
+F 5 "EKZN201ELL561MJ20S" H 700 700 50  0001 C CNN "PartNumber"
+F 6 "200V, 2.75A, 18x20" H 500 400 60  0001 C CNN "Remarks"
 	1    4100 2500
 	1    0    0    -1
@@
 AR Path="/58A68DC9/5D8EDFC0" Ref="R17"  Part="1"
 F 0 "R17" V 2925 6500 50  0000 C CNN
-F 1 "100k" V 3075 6500 50  0000 C CNN
+F 1 "180k" V 3075 6500 50  0000 C CNN
 F 2 "LibreSolar:R_0603_1608" V 2825 6400 50  0001 C CNN
 F 3 "" H 3000 6500 50  0000 C CNN
-F 4 "any" H -3450 1200 50  0001 C CNN "Manufacturer"
-F 5 "" H -3450 1200 50  0001 C CNN "PartNumber"
+F 4 "Yageo" H -3450 1200 50  0001 C CNN "Manufacturer"
+F 5 "RC0603FR-07180KL" H -3450 1200 50  0001 C CNN "PartNumber"
 F 6 "1%" H 3000 6500 50  0001 C CNN "Remarks"
 	1    3000 6500
@@
 AR Path="/58A68DC9/5D8EDFC8" Ref="R18"  Part="1"
 F 0 "R18" V 2925 6900 50  0000 C CNN
-F 1 "5.6k" V 3075 6900 50  0000 C CNN
+F 1 "10k" V 3075 6900 50  0000 C CNN
 F 2 "LibreSolar:R_0603_1608" V 2825 6800 50  0001 C CNN
 F 3 "" H 3000 6900 50  0000 C CNN
-F 4 "any" H -3450 1100 50  0001 C CNN "Manufacturer"
-F 5 "" H -3450 1100 50  0001 C CNN "PartNumber"
+F 4 "Yageo" H -3450 1100 50  0001 C CNN "Manufacturer"
+F 5 "RC0603FR-0710KL" H -3450 1100 50  0001 C CNN "PartNumber"
 F 6 "1%" H 3000 6900 50  0001 C CNN "Remarks"
 	1    3000 6900
@@
 AR Path="/58A68DC9/5D8EDFB8" Ref="R13"  Part="1"
 F 0 "R13" V 1625 5700 50  0000 C CNN
-F 1 "100k" V 1775 5700 50  0000 C CNN
+F 1 "470k" V 1775 5700 50  0000 C CNN
 F 2 "LibreSolar:R_0603_1608" V 1525 5600 50  0001 C CNN
 F 3 "" H 1700 5700 50  0000 C CNN
-F 4 "any" H -5950 400 50  0001 C CNN "Manufacturer"
-F 5 "" H -5950 400 50  0001 C CNN "PartNumber"
+F 4 "Yageo" H -5950 400 50  0001 C CNN "Manufacturer"
+F 5 "RC0603FR-07470KL" H -5950 400 50  0001 C CNN "PartNumber"
 F 6 "1%" H 1700 5700 50  0001 C CNN "Remarks"
 	1    1700 5700
@@
 AR Path="/58A68DC9/5D8EDFB0" Ref="R14"  Part="1"
 F 0 "R14" V 1625 6100 50  0000 C CNN
-F 1 "2.2k" V 1775 6100 50  0000 C CNN
+F 1 "10k" V 1775 6100 50  0000 C CNN
 F 2 "LibreSolar:R_0603_1608" V 1525 6000 50  0001 C CNN
 F 3 "" H 1700 6100 50  0000 C CNN
-F 4 "any" H -5950 300 50  0001 C CNN "Manufacturer"
-F 5 "" H -5950 300 50  0001 C CNN "PartNumber"
+F 4 "Yageo" H -5950 300 50  0001 C CNN "Manufacturer"
+F 5 "RC0603FR-0710KL" H -5950 300 50  0001 C CNN "PartNumber"
 F 6 "1%" H 1700 6100 50  0001 C CNN "Remarks"
 	1    1700 6100
@@
 F 2 "Capacitor_THT:C_Rect_L7.2mm_W3.5mm_P5.00mm_FKS2_FKP2_MKS2_MKP2" H 8500 2800 50  0001 C CNN
 F 3 "" H 8525 3075 50  0001 C CNN
-F 4 "B32529C224J" H 8500 3000 50  0001 C CNN "PartNumber"
-F 5 "EPCOS / TDK" H 8500 3000 50  0001 C CNN "Manufacturer"
-F 6 "Alternative: Kemet MMK5224K63J01L16.5TA18" H 8500 3000 50  0001 C CNN "Remarks"
+F 4 "R463W322050M2M" H 8500 3000 50  0001 C CNN "PartNumber"
+F 5 "WIMA" H 8500 3000 50  0001 C CNN "Manufacturer"
+F 6 "0.22µF, 250V, film" H 8500 3000 50  0001 C CNN "Remarks"
 	1    8500 3000
 	1    0    0    -1
@@
 AR Path="/58A68DC9/5EBC12C9" Ref="RV2"  Part="1"
 F 0 "RV2" H 1803 2296 50  0000 L CNN
-F 1 "82V" H 1803 2205 50  0000 L CNN
+F 1 "150V" H 1803 2205 50  0000 L CNN
 F 2 "Varistor:RV_Disc_D12mm_W4.3mm_P7.5mm" V 1630 2250 50  0001 C CNN
 F 3 "" H 1700 2250 50  0001 C CNN
-F 4 "Bourns" H 1700 2250 50  0001 C CNN "Manufacturer"
-F 5 "MOV-10D820K " H 1700 2250 50  0001 C CNN "PartNumber"
+F 4 "Littelfuse" H 1700 2250 50  0001 C CNN "Manufacturer"
+F 5 "V150LA20AP" H 1700 2250 50  0001 C CNN "PartNumber"
 	1    1700 2250
 	1    0    0    -1
@@
 F 2 "Capacitor_THT:C_Rect_L7.2mm_W3.5mm_P5.00mm_FKS2_FKP2_MKS2_MKP2" H 9100 2800 50  0001 C CNN
 F 3 "" H 9125 3075 50  0001 C CNN
-F 4 "B32529C224J" H 9100 3000 50  0001 C CNN "PartNumber"
-F 5 "EPCOS / TDK" H 9100 3000 50  0001 C CNN "Manufacturer"
-F 6 "Alternative: Kemet MMK5224K63J01L16.5TA18" H 9100 3000 50  0001 C CNN "Remarks"
+F 4 "R463W322050M2M" H 9100 3000 50  0001 C CNN "PartNumber"
+F 5 "WIMA" H 9100 3000 50  0001 C CNN "Manufacturer"
+F 6 "0.22µF, 250V, film" H 9100 3000 50  0001 C CNN "Remarks"
 	1    9100 3000
 	-1   0    0    1
@@
 AR Path="/58A68DC9/5FFA2979" Ref="C27"  Part="1"
 F 0 "C27" H 9920 3070 50  0000 L CNN
-F 1 "680µF" H 9920 2920 50  0000 L CNN
-F 2 "Capacitor_THT:CP_Radial_D10.0mm_P5.00mm" H 9900 3000 50  0001 C CNN
+F 1 "1000µF" H 9920 2920 50  0000 L CNN
+F 2 "Capacitor_THT:CP_Radial_D16.0mm_P7.50mm" H 9900 3000 50  0001 C CNN
 F 3 "" H 9900 3000 50  0000 C CNN
 F 4 "Panasonic" H 6100 1200 50  0001 C CNN "Manufacturer"
-F 5 "EEU-FR1V681" H 6100 1200 50  0001 C CNN "PartNumber"
-F 6 "35V, 2.18A, 10x20" H 1900 200 60  0001 C CNN "Remarks"
+F 5 "EKMQ101VSN102MR40S" H 6100 1200 50  0001 C CNN "PartNumber"
+F 6 "100V, 2.0A, 16x40" H 1900 200 60  0001 C CNN "Remarks"
 	1    9900 3000
 	1    0    0    -1
@@
 	8100 5500 7900 5500
 Text Notes 7600 1300 0    50   ~ 0
-Main inductor L1 layout:\n- Core: 2x stacked MS-130060-2 (Sendust 60µ, OD 33 mm, AL 61 nH/T²)\n- Winding: 21 turns, 40 strands x AWG 27 (D 0.355 mm), 4 mm² total
+Inductor L1 (Bourns SRR1260-470M):\n- 47µH, 50A saturation, 1.8mΩ DCR\n- 12.7×12.7×6mm SMD package\n- High-side MOSFETs Q1, Q2: 2× IPP200N25N3G per position (Q1A||Q1B, Q2A||Q2B)\n- Low-side sync MOSFETs Q4, Q5, Q6: 3× IPP200N25N3G in parallel\n- Gate driver U1: IR2104 half-bridge with bootstrap; 500ns dead-time
 $EndSCHEMATC

Commit message: Implement 1kW hardware upgrade: update component values in KiCad schematics and firmware constants
Co-authored-by: intrinsicaly <43327040+intrinsicaly@users.noreply.github.com>
Parts:
- C2: value 560µF -> 100µF; footprint Capacitor_THT:CP_Radial_D18.0mm_P7.50mm -> Capacitor_THT:CP_Radial_D16.0mm_P7.50mm; Manufacturer United Chemi-Con -> Nichicon; PartNumber EKZN201ELL561MJ20S -> UHE2C101MED; Remarks 200V, 2.75A, 18x20 -> 160V, 2.75A, 16x25; install 4 in parallel (C2a-C2d)
- C27, C5: value 1000µF -> 680µF; footprint Capacitor_THT:CP_Radial_D16.0mm_P7.50mm -> Capacitor_THT:CP_Radial_D18.0mm_P7.50mm; PartNumber EKMQ101VSN102MR40S -> EEEFK1J681P; Remarks 100V, 2.0A, 16x40 -> 63V, 3.97A, 18x20
- L1: value 47µH -> 4.7µH; footprint LibreSolar:Inductor_Bourns_SRR1260 -> LibreSolar:Inductor_Wuerth_7443730470; Manufacturer Bourns -> Würth Elektronik; PartNumber SRR1260-470M -> 7443730470
- Q1: value IPP200N25N3G -> IPW60R041P6; footprint LibreSolar:TO-220-3_Horizontal_BottomHeatsink -> LibreSolar:TO-247-3_Horizontal_BottomHeatsink; PartNumber IPP200N25N3G -> IPW60R041P6; Remarks 250V, 34A, 200mΩ, TO-220; parallel pair Q1A||Q1B -> 650V, 38A, 41mΩ, TO-247; high-side switch
- Q2: value IPP200N25N3G -> IPT015N10N5; PartNumber IPP200N25N3G -> IPT015N10N5; Remarks 250V, 34A, 200mΩ, TO-220; parallel pair Q2A||Q2B -> 100V, 100A, 1.5mΩ, TO-220; low-side synchronous switch
- R13: value 470k -> 499k; PartNumber RC0603FR-07470KL -> RC0603FR-07499KL; Remarks 1% -> 1%; series with R13b (499k) for 140V PV range
- R14: value 10k -> 20k; PartNumber RC0603FR-0710KL -> RC0603FR-0720KL
- R17: value 180k -> 169k; PartNumber RC0603FR-07180KL -> RC0603FR-07169KL
- R6: value 2m -> 1m; PartNumber CRE2512-FZ-R002E-3 -> CRE2512-FZ-R001E-3
- U1: value IR2104 -> UCC27712; Manufacturer Infineon -> Texas Instruments; PartNumber IR2104STRPBF -> UCC27712DR
- U3: value INA186 -> INA240A3; PartNumber INA186A1IDCKR -> INA240A3DCNR
Other:
- note added: "Inductor L1 (Würth 7443730470):\n- 4.7µH, 50A saturation, 2.4mΩ DCR\n- 22.5×22.5×19.5mm radial through-hole\n- High-side MOSFET Q1: IPW60R041P6 (650V, 38A, 41mΩ, TO-247)\n- Low-side MOSFET Q2: IPT015N10N5 (100V, 100A, 1.5mΩ, TO-220)\n- Gate driver U1: UCC27712 half-bridge, 150V bootstrap; 500ns dead-time"
- note removed: "Inductor L1 (Bourns SRR1260-470M):\n- 47µH, 50A saturation, 1.8mΩ DCR\n- 12.7×12.7×6mm SMD package\n- High-side MOSFETs Q1, Q2: 2× IPP200N25N3G per position (Q1A||Q1B, Q2A||Q2B)\n- Low-side sync MOSFETs Q4, Q5, Q6: 3× IPP200N25N3G in parallel\n- Gate driver U1: IR2104 half-bridge with bootstrap; 500ns dead-time"
Changed lines of the file:
@@
 AR Path="/58A68DC9/58ACD441" Ref="L1"  Part="1"
 F 0 "L1" V 8250 2500 50  0000 C CNN
-F 1 "47µH" V 8075 2500 50  0000 C CNN
-F 2 "LibreSolar:Inductor_Bourns_SRR1260" V 8350 2500 50  0001 C CNN
+F 1 "4.7µH" V 8075 2500 50  0000 C CNN
+F 2 "LibreSolar:Inductor_Wuerth_7443730470" V 8350 2500 50  0001 C CNN
 F 3 "" H 8150 2500 50  0001 C CNN
-F 4 "Bourns" H 750 450 50  0001 C CNN "Manufacturer"
-F 5 "SRR1260-470M" H 8150 2500 60  0001 C CNN "PartNumber"
+F 4 "Würth Elektronik" H 750 450 50  0001 C CNN "Manufacturer"
+F 5 "7443730470" H 8150 2500 60  0001 C CNN "PartNumber"
 	1    8150 2500
 	0    -1   -1   0
@@
 AR Path="/58A68DC9/58A857B0" Ref="C2"  Part="1"
 F 0 "C2" H 4525 2575 50  0000 L CNN
-F 1 "560µF" H 4525 2425 50  0000 L CNN
-F 2 "Capacitor_THT:CP_Radial_D18.0mm_P7.50mm" H 4525 2275 50  0001 L CNN
+F 1 "100µF" H 4525 2425 50  0000 L CNN
+F 2 "Capacitor_THT:CP_Radial_D16.0mm_P7.50mm" H 4525 2275 50  0001 L CNN
 F 3 "" H 4525 2575 50  0000 C CNN
-F 4 "United Chemi-Con" H 1100 700 50  0001 C CNN "Manufacturer"
-F 5 "EKZN201ELL561MJ20S" H 1100 700 50  0001 C CNN "PartNumber"
-F 6 "200V, 2.75A, 18x20" H 500 400 60  0001 C CNN "Remarks"
+F 4 "Nichicon" H 1100 700 50  0001 C CNN "Manufacturer"
+F 5 "UHE2C101MED" H 1100 700 50  0001 C CNN "PartNumber"
+F 6 "160V, 2.75A, 16x25; install 4 in parallel (C2a-C2d)" H 500 400 60  0001 C CNN "Remarks"
 	1    4500 2500
 	1    0    0    -1
@@
 AR Path="/58A68DC9/5EBC12A8" Ref="C5"  Part="1"
 F 0 "C5" H 9520 3070 50  0000 L CNN
-F 1 "1000µF" H 9520 2920 50  0000 L CNN
-F 2 "Capacitor_THT:CP_Radial_D16.0mm_P7.50mm" H 9500 3000 50  0001 C CNN
+F 1 "680µF" H 9520 2920 50  0000 L CNN
+F 2 "Capacitor_THT:CP_Radial_D18.0mm_P7.50mm" H 9500 3000 50  0001 C CNN
 F 3 "" H 9500 3000 50  0000 C CNN
 F 4 "Panasonic" H 5700 1200 50  0001 C CNN "Manufacturer"
-F 5 "EKMQ101VSN102MR40S" H 5700 1200 50  0001 C CNN "PartNumber"
-F 6 "100V, 2.0A, 16x40" H 1500 200 60  0001 C CNN "Remarks"
+F 5 "EEEFK1J681P" H 5700 1200 50  0001 C CNN "PartNumber"
+F 6 "63V, 3.97A, 18x20" H 1500 200 60  0001 C CNN "Remarks"
 	1    9500 3000
 	1    0    0    -1
@@
 P 8700 5500
 F 0 "U1" H 8700 5850 50  0000 C CNN
-F 1 "IR2104" H 8700 5150 50  0000 C CNN
+F 1 "UCC27712" H 8700 5150 50  0000 C CNN
 F 2 "LibreSolar:SOIC-8_3.9x4.9mm_Pitch1.27mm" H 8750 5500 60  0001 C CNN
 F 3 "" H 8750 5500 60  0001 C CNN
-F 4 "Infineon" H 4500 1450 50  0001 C CNN "Manufacturer"
-F 5 "IR2104STRPBF" H 4500 1450 50  0001 C CNN "PartNumber"
+F 4 "Texas Instruments" H 4500 1450 50  0001 C CNN "Manufacturer"
+F 5 "UCC27712DR" H 4500 1450 50  0001 C CNN "PartNumber"
 	1    8700 5500
 	1    0    0    -1
@@
 P 6900 2100
 F 0 "Q1" H 7100 2150 50  0000 L CNN
-F 1 "IPP200N25N3G" H 7100 2050 50  0000 L CNN
-F 2 "LibreSolar:TO-220-3_Horizontal_BottomHeatsink" H 7100 2200 50  0001 C CNN
+F 1 "IPW60R041P6" H 7100 2050 50  0000 L CNN
+F 2 "LibreSolar:TO-247-3_Horizontal_BottomHeatsink" H 7100 2200 50  0001 C CNN
 F 3 "" H 6900 2100 50  0001 C CNN
 F 4 "Infineon" H 900 300 50  0001 C CNN "Manufacturer"
-F 5 "IPP200N25N3G" H 900 300 50  0001 C CNN "PartNumber"
+F 5 "IPW60R041P6" H 900 300 50  0001 C CNN "PartNumber"
 F 6 "" H 6900 2100 50  0001 C CNN "Alternative"
-F 7 "250V, 34A, 200mΩ, TO-220; parallel pair Q1A||Q1B" H 6900 2100 50  0001 C CNN "Remarks"
+F 7 "650V, 38A, 41mΩ, TO-247; high-side switch" H 6900 2100 50  0001 C CNN "Remarks"
 	1    6900 2100
 	1    0    0    -1
@@
 P 6900 3000
 F 0 "Q2" H 7100 3050 50  0000 L CNN
-F 1 "IPP200N25N3G" H 7100 2950 50  0000 L CNN
+F 1 "IPT015N10N5" H 7100 2950 50  0000 L CNN
 F 2 "LibreSolar:TO-220-3_Horizontal_BottomHeatsink" H 7100 3100 50  0001 C CNN
 F 3 "" H 6900 3000 50  0001 C CNN
 F 4 "Infineon" H 900 500 50  0001 C CNN "Manufacturer"
-F 5 "IPP200N25N3G" H 900 500 50  0001 C CNN "PartNumber"
+F 5 "IPT015N10N5" H 900 500 50  0001 C CNN "PartNumber"
 F 6 "" H 6900 3000 50  0001 C CNN "Alternative"
-F 7 "250V, 34A, 200mΩ, TO-220; parallel pair Q2A||Q2B" H 6900 3000 50  0001 C CNN "Remarks"
+F 7 "100V, 100A, 1.5mΩ, TO-220; low-side synchronous switch" H 6900 3000 50  0001 C CNN "Remarks"
 	1    6900 3000
 	1    0    0    -1
@@
 AR Path="/5C45ED62/5C59CE9B" Ref="R?"  Part="1"
 F 0 "R6" V 8730 2500 50  0000 C CNN
-F 1 "2m" V 8870 2500 50  0000 C CNN
+F 1 "1m" V 8870 2500 50  0000 C CNN
 F 2 "LibreSolar:R_Bourns_CRE2512" H 8800 2500 50  0001 C CNN
 F 3 "" H 8800 2500 50  0000 C CNN
 F 4 "Bourns" H 7050 -3400 50  0001 C CNN "Manufacturer"
-F 5 "CRE2512-FZ-R002E-3" H 7050 -3400 50  0001 C CNN "PartNumber"
+F 5 "CRE2512-FZ-R001E-3" H 7050 -3400 50  0001 C CNN "PartNumber"
 	1    8800 2500
 	0    1    1    0
@@
 AR Path="/58A68DC9/5D8EDFC0" Ref="R17"  Part="1"
 F 0 "R17" V 2925 6500 50  0000 C CNN
-F 1 "180k" V 3075 6500 50  0000 C CNN
+F 1 "169k" V 3075 6500 50  0000 C CNN
 F 2 "LibreSolar:R_0603_1608" V 2825 6400 50  0001 C CNN
 F 3 "" H 3000 6500 50  0000 C CNN
 F 4 "Yageo" H -3450 1200 50  0001 C CNN "Manufacturer"
-F 5 "RC0603FR-07180KL" H -3450 1200 50  0001 C CNN "PartNumber"
+F 5 "RC0603FR-07169KL" H -3450 1200 50  0001 C CNN "PartNumber"
 F 6 "1%" H 3000 6500 50  0001 C CNN "Remarks"
 	1    3000 6500
@@
 AR Path="/58A68DC9/5D8EDFB8" Ref="R13"  Part="1"
 F 0 "R13" V 1625 5700 50  0000 C CNN
-F 1 "470k" V 1775 5700 50  0000 C CNN
+F 1 "499k" V 1775 5700 50  0000 C CNN
 F 2 "LibreSolar:R_0603_1608" V 1525 5600 50  0001 C CNN
 F 3 "" H 1700 5700 50  0000 C CNN
 F 4 "Yageo" H -5950 400 50  0001 C CNN "Manufacturer"
-F 5 "RC0603FR-07470KL" H -5950 400 50  0001 C CNN "PartNumber"
-F 6 "1%" H 1700 5700 50  0001 C CNN "Remarks"
+F 5 "RC0603FR-07499KL" H -5950 400 50  0001 C CNN "PartNumber"
+F 6 "1%; series with R13b (499k) for 140V PV range" H 1700 5700 50  0001 C CNN "Remarks"
 	1    1700 5700
 	1    0    0    -1
@@
 AR Path="/58A68DC9/5D8EDFB0" Ref="R14"  Part="1"
 F 0 "R14" V 1625 6100 50  0000 C CNN
-F 1 "10k" V 1775 6100 50  0000 C CNN
+F 1 "20k" V 1775 6100 50  0000 C CNN
 F 2 "LibreSolar:R_0603_1608" V 1525 6000 50  0001 C CNN
 F 3 "" H 1700 6100 50  0000 C CNN
 F 4 "Yageo" H -5950 300 50  0001 C CNN "Manufacturer"
-F 5 "RC0603FR-0710KL" H -5950 300 50  0001 C CNN "PartNumber"
+F 5 "RC0603FR-0720KL" H -5950 300 50  0001 C CNN "PartNumber"
 F 6 "1%" H 1700 6100 50  0001 C CNN "Remarks"
 	1    1700 6100
@@
 AR Path="/58A68DC9/5EE3E924" Ref="U3"  Part="1"
 F 0 "U3" H 5550 5650 50  0000 L CNN
-F 1 "INA186" H 5550 5550 50  0000 L CNN
+F 1 "INA240A3" H 5550 5550 50  0000 L CNN
 F 2 "Package_TO_SOT_SMD:SOT-363_SC-70-6" H 5550 5350 50  0001 C CNN
-F 3 "http://www.ti.com/lit/ds/symlink/ina186.pdf" H 5650 5450 50  0001 C CNN
+F 3 "http://www.ti.com/lit/ds/symlink/ina240.pdf" H 5650 5450 50  0001 C CNN
 F 4 "Texas Instruments" H 5500 5300 50  0001 C CNN "Manufacturer"
-F 5 "INA186A1IDCKR" H 5500 5300 50  0001 C CNN "PartNumber"
+F 5 "INA240A3DCNR" H 5500 5300 50  0001 C CNN "PartNumber"
 	1    5500 5300
 	1    0    0    -1
@@
 AR Path="/58A68DC9/5FFA2979" Ref="C27"  Part="1"
 F 0 "C27" H 9920 3070 50  0000 L CNN
-F 1 "1000µF" H 9920 2920 50  0000 L CNN
-F 2 "Capacitor_THT:CP_Radial_D16.0mm_P7.50mm" H 9900 3000 50  0001 C CNN
+F 1 "680µF" H 9920 2920 50  0000 L CNN
+F 2 "Capacitor_THT:CP_Radial_D18.0mm_P7.50mm" H 9900 3000 50  0001 C CNN
 F 3 "" H 9900 3000 50  0000 C CNN
 F 4 "Panasonic" H 6100 1200 50  0001 C CNN "Manufacturer"
-F 5 "EKMQ101VSN102MR40S" H 6100 1200 50  0001 C CNN "PartNumber"
-F 6 "100V, 2.0A, 16x40" H 1900 200 60  0001 C CNN "Remarks"
+F 5 "EEEFK1J681P" H 6100 1200 50  0001 C CNN "PartNumber"
+F 6 "63V, 3.97A, 18x20" H 1900 200 60  0001 C CNN "Remarks"
 	1    9900 3000
 	1    0    0    -1
@@
 	8100 5500 7900 5500
 Text Notes 7600 1300 0    50   ~ 0
-Inductor L1 (Bourns SRR1260-470M):\n- 47µH, 50A saturation, 1.8mΩ DCR\n- 12.7×12.7×6mm SMD package\n- High-side MOSFETs Q1, Q2: 2× IPP200N25N3G per position (Q1A||Q1B, Q2A||Q2B)\n- Low-side sync MOSFETs Q4, Q5, Q6: 3× IPP200N25N3G in parallel\n- Gate driver U1: IR2104 half-bridge with bootstrap; 500ns dead-time
+Inductor L1 (Würth 7443730470):\n- 4.7µH, 50A saturation, 2.4mΩ DCR\n- 22.5×22.5×19.5mm radial through-hole\n- High-side MOSFET Q1: IPW60R041P6 (650V, 38A, 41mΩ, TO-247)\n- Low-side MOSFET Q2: IPT015N10N5 (100V, 100A, 1.5mΩ, TO-220)\n- Gate driver U1: UCC27712 half-bridge, 150V bootstrap; 500ns dead-time
 $EndSCHEMATC
