File: kicad/dcdc.sch (KiCad schematic (older format))
At the start: 51 parts, among them Q1 IPW60R041P6, Q2 IPT015N10N5, Q3 IPA045N10N3G, U1 UCC27712, U3 INA240A3

Commit message: Sync KiCad PCB to updated power stage
Parts:
- C2: footprint Capacitor_THT:CP_Radial_D16.0mm_P7.50mm -> Capacitor_THT:CP_Radial_D18.0mm_P7.50mm
- C27, C5: footprint Capacitor_THT:CP_Radial_D18.0mm_P7.50mm -> Project:CP_Radial_D18.0mm_P5.00mm_Adapted
- L1: footprint LibreSolar:Inductor_Wuerth_7443730470 -> Project:Inductor_4p7uH_HighCurrent_ToroidPad
- Q1: footprint LibreSolar:TO-247-3_Horizontal_BottomHeatsink -> Project:TO-247-3_Horizontal_BottomHeatsink_Adapted
Changed lines of the file:
@@
 F 0 "L1" V 8250 2500 50  0000 C CNN
 F 1 "4.7µH" V 8075 2500 50  0000 C CNN
-F 2 "LibreSolar:Inductor_Wuerth_7443730470" V 8350 2500 50  0001 C CNN
+F 2 "Project:Inductor_4p7uH_HighCurrent_ToroidPad" V 8350 2500 50  0001 C CNN
 F 3 "" H 8150 2500 50  0001 C CNN
 F 4 "Würth Elektronik" H 750 450 50  0001 C CNN "Manufacturer"
@@
 F 0 "C2" H 4525 2575 50  0000 L CNN
 F 1 "100µF" H 4525 2425 50  0000 L CNN
-F 2 "Capacitor_THT:CP_Radial_D16.0mm_P7.50mm" H 4525 2275 50  0001 L CNN
+F 2 "Capacitor_THT:CP_Radial_D18.0mm_P7.50mm" H 4525 2275 50  0001 L CNN
 F 3 "" H 4525 2575 50  0000 C CNN
 F 4 "Nichicon" H 1100 700 50  0001 C CNN "Manufacturer"
@@
 F 0 "C5" H 9520 3070 50  0000 L CNN
 F 1 "680µF" H 9520 2920 50  0000 L CNN
-F 2 "Capacitor_THT:CP_Radial_D18.0mm_P7.50mm" H 9500 3000 50  0001 C CNN
+F 2 "Project:CP_Radial_D18.0mm_P5.00mm_Adapted" H 9500 3000 50  0001 C CNN
 F 3 "" H 9500 3000 50  0000 C CNN
 F 4 "Panasonic" H 5700 1200 50  0001 C CNN "Manufacturer"
@@
 F 0 "Q1" H 7100 2150 50  0000 L CNN
 F 1 "IPW60R041P6" H 7100 2050 50  0000 L CNN
-F 2 "LibreSolar:TO-247-3_Horizontal_BottomHeatsink" H 7100 2200 50  0001 C CNN
+F 2 "Project:TO-247-3_Horizontal_BottomHeatsink_Adapted" H 7100 2200 50  0001 C CNN
 F 3 "" H 6900 2100 50  0001 C CNN
 F 4 "Infineon" H 900 300 50  0001 C CNN "Manufacturer"
@@
 F 0 "C27" H 9920 3070 50  0000 L CNN
 F 1 "680µF" H 9920 2920 50  0000 L CNN
-F 2 "Capacitor_THT:CP_Radial_D18.0mm_P7.50mm" H 9900 3000 50  0001 C CNN
+F 2 "Project:CP_Radial_D18.0mm_P5.00mm_Adapted" H 9900 3000 50  0001 C CNN
 F 3 "" H 9900 3000 50  0000 C CNN
 F 4 "Panasonic" H 6100 1200 50  0001 C CNN "Manufacturer"
