File: kicad/can.sch (KiCad schematic (older format))
At the start: 11 parts, among them U5 TCAN334

Commit message: Align docs and firmware with 24V/48V baseline
Other:
- note added: "CAN bus power supply\n- 24V-58V\n- 600 mA (like PoE)\n\nDiodes necessary to prevent\nseparate GND loops.\n\nPolyfuse to prevent \nover-current in daisy-chained \nbus with multiple sources and \nsinks."
- note removed: "CAN bus power supply\n- 10V-32V\n- 600 mA (like PoE)\n\nDiodes necessary to prevent\nseparate GND loops.\n\nPolyfuse to prevent \nover-current in daisy-chained \nbus with multiple sources and \nsinks."
Changed lines of the file:
@@
 Connection ~ 6900 2900
 Text Notes 8000 5100 0    50   ~ 0
-CAN bus power supply\n- 10V-32V\n- 600 mA (like PoE)\n\nDiodes necessary to prevent\nseparate GND loops.\n\nPolyfuse to prevent \nover-current in daisy-chained \nbus with multiple sources and \nsinks.
+CAN bus power supply\n- 24V-58V\n- 600 mA (like PoE)\n\nDiodes necessary to prevent\nseparate GND loops.\n\nPolyfuse to prevent \nover-current in daisy-chained \nbus with multiple sources and \nsinks.
 Text HLabel 7600 2900 2    50   Output ~ 0
 CAN_PWR1

Commit message: Address review follow-ups and portability issues
Other:
- note added: "CAN bus power supply\n- 24V/48V battery systems\n- bus voltage up to 58V\n- 600 mA (like PoE)\n\nDiodes necessary to prevent\nseparate GND loops.\n\nPolyfuse to prevent \nover-current in daisy-chained \nbus with multiple sources and \nsinks."
- note removed: "CAN bus power supply\n- 24V-58V\n- 600 mA (like PoE)\n\nDiodes necessary to prevent\nseparate GND loops.\n\nPolyfuse to prevent \nover-current in daisy-chained \nbus with multiple sources and \nsinks."
Changed lines of the file:
@@
 Connection ~ 6900 2900
 Text Notes 8000 5100 0    50   ~ 0
-CAN bus power supply\n- 24V-58V\n- 600 mA (like PoE)\n\nDiodes necessary to prevent\nseparate GND loops.\n\nPolyfuse to prevent \nover-current in daisy-chained \nbus with multiple sources and \nsinks.
+CAN bus power supply\n- 24V/48V battery systems\n- bus voltage up to 58V\n- 600 mA (like PoE)\n\nDiodes necessary to prevent\nseparate GND loops.\n\nPolyfuse to prevent \nover-current in daisy-chained \nbus with multiple sources and \nsinks.
 Text HLabel 7600 2900 2    50   Output ~ 0
 CAN_PWR1
