File: kicad/mppt-4820-hc.kicad_pcb (KiCad board)
At the start: 4 copper layers, 100 x 100 mm, 172 parts, among them J1 MKDS 5/ 2-9,5, J2 MKDS 5/ 2-9,5, J3 MKDS 5/ 2-9,5, J4 8P8C, J5 8P8C, J6 JST PH, J7 UEXT, P1 CONN_01X02, Q1 IPA045N10N3G, Q2 IPA045N10N3G, Q3 IPA045N10N3G, Q4 BUK98180-100A, Q7 IPA045N10N3G, T1 BC846B, T10 BC846B, T2 BC846B, T3 BC846B, T4 BC856B, T5 BC846B, U1 LM5107, U2 STM32G431CBTx, U3 INA186, U4 LMR16006X, U5 INA186, U6 W25Q80DVS, U7 TCAN334, Y1 8MHz

Commit message: Sync KiCad PCB to updated power stage
Parts:
- C1: value 390µF -> 560µF
- C2: value 390µF -> 100µF
- C27, C5: footprint Capacitor_THT:CP_Radial_D10.0mm_P5.00mm -> Project:CP_Radial_D18.0mm_P5.00mm_Adapted
- L1: value 53µH -> 4.7µH; footprint LibreSolar:Inductor_Toroid_D32.8mm_4mm2 -> Project:Inductor_4p7uH_HighCurrent_ToroidPad
- Q1: value IPA045N10N3G -> IPW60R041P6; footprint LibreSolar:TO-220-3_Horizontal_BottomHeatsink -> Project:TO-247-3_Horizontal_BottomHeatsink_Adapted
- Q2: value IPA045N10N3G -> IPT015N10N5
- R13: value 100k -> 499k
- R14: value 2.2k -> 20k
- R17: value 100k -> 169k
- R18: value 5.6k -> 10k
- R6: value 2m -> 1m
- RV2: value 82V -> 150V
- U1: value LM5107 -> UCC27712
- U3: value INA186 -> INA240A3
- U4: value LMR16006X -> LMR16030X
Other:
- net class Default: clearance 0.2 -> 0.25; via_dia 0.7 -> 0.8; via_drill 0.3 -> 0.4
- net class HV_48V added: clearance 0.5, trace_width 1, via_dia 1, via_drill 0.5
- net class HighCurrent_20A added: clearance 0.4, trace_width 1.5, via_dia 1, via_drill 0.5
- net class HighCurrent_42A added: clearance 0.5, trace_width 2, via_dia 1.2, via_drill 0.6
- net class Power: clearance 0.2 -> 0.25; trace_width 0.4 -> 0.6
- rule trace_clearance: 0.2 -> 0.3
- rule via_min_size: 0.3 -> 0.6
